File: Numpad2.kicad_pcb (KiCad board)
At the start: 2 copper layers, 104.8 x 82 mm, 93 parts, among them U1 RP2040-ZERO, U2 SN74LV1T34DBVR

Commit message: Add files via upload
Parts:
- added C20: 100nF, Capacitor_SMD:C_0402_1005Metric_Pad0.74x0.62mm_HandSolder, B.Cu at (190.5, 119.4)
- added C21: 100nF, Capacitor_SMD:C_0402_1005Metric_Pad0.74x0.62mm_HandSolder, B.Cu at (190.5, 138.4)
- added D17: 1N4148WS, Numpad:D_SOD-323, B.Cu at (194.5, 128.6)
- added D18: 1N4148WS, Numpad:D_SOD-323, B.Cu at (194.5, 109.7)
- added H1: MountingHole_Pad, Numpad:MountingHole_2.2mm_M2_Pad, F.Cu at (118.2, 65.8)
- added H2: MountingHole_Pad, Numpad:MountingHole_2.2mm_M2_Pad, F.Cu at (88.0, 88.8)
- added H3: MountingHole_Pad, Numpad:MountingHole_2.2mm_M2_Pad, F.Cu at (88.0, 94.8)
- added H4: MountingHole_Pad, Numpad:MountingHole_2.2mm_M2_Pad, F.Cu at (88.0, 100.8)
- added K_LED15: SK6812-E, Numpad:LED_SK6812-E, B.Cu at (185.6, 119.1)
- added K_LED16: SK6812-E, Numpad:LED_SK6812-E, B.Cu at (185.6, 138.2)
- added R15: 27, Resistor_SMD:R_0402_1005Metric_Pad0.72x0.64mm_HandSolder, B.Cu at (191.0, 92.5)
- added Sw16: ~, PCM_Switch_Keyboard_Hotswap_Kailh:SW_Hotswap_Kailh_MX, F.Cu at (185.6, 133.2)
- added Sw17: ~, PCM_Switch_Keyboard_Hotswap_Kailh:SW_Hotswap_Kailh_MX, F.Cu at (185.6, 114.1)
- C1, C2, C3: value 100nF -> 10nF; moved to B.Cu
- C10, C11, C12, C13, C14, C15, C16, C17, C18, C19, C4, C5, C6, C7, C8, C9, R10, R11, R12, R9, TP1, TP2, TP3, TP4, TP5, TP6, TP9, U2: moved to B.Cu
- U1: moved to F.Cu
- moved C16 96.0 mm to (190.2, 157.4), turned to 90 degrees
- moved TP5 95.3 mm to (196.8, 83.4), turned to 180 degrees
- moved TP3 88.3 mm to (190.1, 78.8), turned to 180 degrees
- moved TP7 87.5 mm to (194.7, 90.9)
- moved D32 86.9 mm to (156.2, 66.0), turned to 0 degrees
- moved TP6 84.4 mm to (188.7, 71.3), turned to 180 degrees
- moved TP9 84.3 mm to (191.7, 102.1), turned to 180 degrees
- moved TP10 81.6 mm to (188.9, 104.2)
- moved TP4 81.3 mm to (182.7, 81.2), turned to 180 degrees
- moved C12 80.6 mm to (171.4, 157.4), turned to 90 degrees
- moved D1 79.7 mm to (137.2, 147.7), turned to -90 degrees
- moved Sw1 79.7 mm to (128.4, 152.2)
- moved K_LED0 79.5 mm to (128.3, 157.0), turned to 0 degrees
- moved TP2 78.8 mm to (180.2, 75.7), turned to 180 degrees
- moved C8 78.5 mm to (152.4, 157.3), turned to 90 degrees
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Connections:
- C1 pad 1: +5V -> +3V3
- D1 pad 1: /ROW0 -> /ROW4
- D13 pad 1: /ROW3 -> /ROW4
- D5 pad 1: /ROW1 -> /ROW4
- D9 pad 1: /ROW2 -> /ROW4
- K_LED0 pad 2: /LED1_IN -> /LED14_IN
- K_LED0 pad 4: /LED0_IN -> /LED13_IN
- K_LED1 pad 2: /LED2_IN -> /LED1_IN
- K_LED1 pad 4: /LED1_IN -> /LED0_IN
- K_LED10 pad 2: /LED11_IN -> /LED8_IN
- K_LED10 pad 4: /LED10_IN -> /LED7_IN
- K_LED11 pad 2: /LED12_IN -> unconnected-(K_LED11-DOUT-Pad2)
- K_LED11 pad 4: /LED11_IN -> /LED16_IN
- K_LED12 pad 2: /LED13_IN -> /LED10_IN
- K_LED12 pad 4: /LED12_IN -> /LED9_IN
- K_LED13 pad 2: /LED14_IN -> /LED11_IN
- K_LED13 pad 4: /LED13_IN -> /LED10_IN
- K_LED14 pad 2: unconnected-(K_LED14-DOUT-Pad2) -> /LED12_IN
- K_LED14 pad 4: /LED14_IN -> /LED11_IN
- K_LED2 pad 2: /LED_3IN -> /LED2_IN
- K_LED2 pad 4: /LED2_IN -> /LED1_IN
- K_LED3 pad 2: /LED4_IN -> /LED15_IN
- K_LED3 pad 4: /LED_3IN -> /LED14_IN
- K_LED4 pad 2: /LED5_IN -> /LED_3IN
- K_LED4 pad 4: /LED4_IN -> /LED2_IN
- K_LED5 pad 2: /LED6_IN -> /LED4_IN
- K_LED5 pad 4: /LED5_IN -> /LED_3IN
- K_LED6 pad 2: /LED7_IN -> /LED5_IN
- K_LED6 pad 4: /LED6_IN -> /LED4_IN
- K_LED7 pad 2: /LED8_IN -> /LED16_IN
- K_LED7 pad 4: /LED7_IN -> /LED15_IN
- K_LED8 pad 2: /LED9_IN -> /LED6_IN
- K_LED8 pad 4: /LED8_IN -> /LED5_IN
- K_LED9 pad 2: /LED10_IN -> /LED7_IN
- K_LED9 pad 4: /LED9_IN -> /LED6_IN
- R1 pad 1: Net-(U1-GP3) -> Net-(U1-GP4)
- R10 pad 1: +5V -> +3V3
- R13 pad 1: Net-(U1-GP14) -> Net-(U1-GP15)
- R2 pad 1: Net-(U1-GP2) -> Net-(U1-GP3)
- R3 pad 1: Net-(U1-GP1) -> Net-(U1-GP2)
- R4 pad 1: Net-(U1-GP0) -> Net-(U1-GP1)
- R9 pad 1: +5V -> +3V3
- Sw10 pad 1: /COL2 -> /COL1
- Sw11 pad 1: /COL3 -> /COL2
- Sw12 pad 1: /COL0 -> /COL3
- Sw13 pad 1: /COL1 -> /COL0
- Sw14 pad 1: /COL2 -> /COL1
- Sw15 pad 1: /COL3 -> /COL2
- Sw2 pad 1: /COL1 -> /COL0
- Sw3 pad 1: /COL2 -> /COL1
- Sw4 pad 1: /COL0 -> /COL1
- Sw5 pad 1: /COL1 -> /COL0
- Sw6 pad 1: /COL2 -> /COL1
- Sw7 pad 1: /COL3 -> /COL2
- Sw8 pad 1: /COL0 -> /COL2
- Sw9 pad 1: /COL1 -> /COL0
- U1 pad 1: Net-(U1-GP0) -> unconnected-(U1-GP0-Pad1)
- U1 pad 16: unconnected-(U1-GP15-Pad16) -> Net-(U1-GP15)
- U1 pad 5: unconnected-(U1-GP4-Pad5) -> Net-(U1-GP4)
Routing:
- net +5V: track 0.00 -> 521.6 mm, vias 0 -> 22
- net /COL0: track 0.00 -> 175.4 mm, vias 0 -> 2
- net /ROW3: track 0.00 -> 156.8 mm, vias 0 -> 6
- net /COL1: track 0.00 -> 155.0 mm, vias 0 -> 2
- net /COL3: track 0.00 -> 141.2 mm, vias 0 -> 5
- net /COL2: track 0.00 -> 123.8 mm, vias 0 -> 2
- net /ROW4: track 0.00 -> 122.0 mm, vias 0 -> 4
- net /LED9_IN: track 0.00 -> 101.7 mm, vias 0 -> 2
- net /LED13_IN: track 0.00 -> 101.3 mm, vias 0 -> 2
- net /LED0_IN: track 0.00 -> 92.8 mm, vias 0 -> 4
- net /LED5_IN: track 0.00 -> 83.6 mm, vias 0 -> 2
- net /ROW2: track 0.00 -> 83.1 mm, vias 0 -> 5
- net /ROW0: track 0.00 -> 81.6 mm, vias 0 -> 6
- net /LED2_IN: track 0.00 -> 65.8 mm, vias 0 -> 2
- net /ROW1: track 0.00 -> 61.3 mm, vias 0 -> 5
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- added copper zone on F.Cu, net GND
Other:
- board size 104.8 x 82 mm -> 86.5 x 101 mm
- board text added: "GND"
- board text added: "Sw6"
- board text added: "Sw7"
