File: Numpad2.kicad_sch (KiCad schematic)
At the start: 98 parts, among them U1 RP2040-ZERO, U2 SN74LV1T34DBVR

Commit message: Add files via upload
Parts:
- added C20, C21: 100nF, Capacitor_SMD:C_0402_1005Metric_Pad0.74x0.62mm_HandSolder, symbol Device:C_Small
- added H1, H2, H3, H4: MountingHole_Pad, Numpad:MountingHole_2.2mm_M2_Pad, symbol Numpad2:MountingHole_Pad
- added K_LED15, K_LED16: SK6812-E, Numpad:LED_SK6812-E, symbol Numpad2:SK6812-E
Connections:
- net +3V3: now also C1.1, R10.1, R9.1
- net +5V: now also C20.1, C21.1, K_LED15.1 (VDD), K_LED16.1 (VDD); no longer C1.1, R10.1, R9.1
- net COL0: now also Sw13.1, Sw2.1, Sw5.1, Sw9.1; no longer Sw12.1, Sw4.1, Sw8.1
- net COL1: now also Sw10.1, Sw14.1, Sw3.1, Sw4.1, Sw6.1; no longer Sw13.1, Sw2.1, Sw5.1, Sw9.1
- net COL2: now also Sw11.1, Sw15.1, Sw7.1, Sw8.1; no longer Sw10.1, Sw14.1, Sw3.1, Sw6.1
- net COL3: now also Sw12.1, Sw16.1, Sw17.1; no longer Sw11.1, Sw15.1, Sw7.1
- net GND: now also C20.2, C21.2, H1.1, H2.1, H3.1, H4.1, K_LED15.3 (GND), K_LED16.3 (GND)
- net LED0_IN: now also K_LED1.4 (DIN); no longer K_LED0.4 (DIN)
- net LED10_IN: now also K_LED12.2 (DOUT), K_LED13.4 (DIN); no longer K_LED10.4 (DIN), K_LED9.2 (DOUT)
- net LED11_IN: now also K_LED13.2 (DOUT), K_LED14.4 (DIN); no longer K_LED10.2 (DOUT), K_LED11.4 (DIN)
- net LED12_IN: now also K_LED14.2 (DOUT), K_LED16.4 (DIN); no longer K_LED11.2 (DOUT), K_LED12.4 (DIN)
- net LED13_IN: now also K_LED0.4 (DIN), K_LED16.2 (DOUT); no longer K_LED12.2 (DOUT), K_LED13.4 (DIN)
- net LED14_IN: now also K_LED0.2 (DOUT), K_LED3.4 (DIN); no longer K_LED13.2 (DOUT), K_LED14.4 (DIN)
- net LED1_IN: now also K_LED1.2 (DOUT), K_LED2.4 (DIN); no longer K_LED0.2 (DOUT), K_LED1.4 (DIN)
- net LED2_IN: now also K_LED2.2 (DOUT), K_LED4.4 (DIN); no longer K_LED1.2 (DOUT), K_LED2.4 (DIN)
- net LED4_IN: now also K_LED5.2 (DOUT), K_LED6.4 (DIN); no longer K_LED3.2 (DOUT), K_LED4.4 (DIN)
- net LED5_IN: now also K_LED6.2 (DOUT), K_LED8.4 (DIN); no longer K_LED4.2 (DOUT), K_LED5.4 (DIN)
- net LED6_IN: now also K_LED8.2 (DOUT), K_LED9.4 (DIN); no longer K_LED5.2 (DOUT), K_LED6.4 (DIN)
- net LED7_IN: now also K_LED10.4 (DIN), K_LED9.2 (DOUT); no longer K_LED6.2 (DOUT), K_LED7.4 (DIN)
- net LED8_IN: now also K_LED10.2 (DOUT), K_LED15.4 (DIN); no longer K_LED7.2 (DOUT), K_LED8.4 (DIN)
- net LED9_IN: now also K_LED12.4 (DIN), K_LED15.2 (DOUT); no longer K_LED8.2 (DOUT), K_LED9.4 (DIN)
- net LED_3IN: now also K_LED4.2 (DOUT), K_LED5.4 (DIN); no longer K_LED2.2 (DOUT), K_LED3.4 (DIN)
- net ROW0: no longer D1.1 (K), D17.1 (K)
- net ROW1: no longer D18.1 (K), D5.1 (K)
- net ROW2: now also D18.1 (K); no longer D9.1 (K)
- net ROW3: now also D17.1 (K); no longer D13.1 (K)
- net at R15.1: now also U1.15 (GP14); no longer U1.1 (GP0)
- net at R13.1: now also U1.16 (GP15); no longer U1.15 (GP14)
- removed net COL4: R15.2, Sw16.1, Sw17.1
- new net LED15_IN: K_LED3.2 (DOUT), K_LED7.4 (DIN)
- new net LED16_IN: K_LED11.4 (DIN), K_LED7.2 (DOUT)
- new net ROW4: D1.1 (K), D13.1 (K), D5.1 (K), D9.1 (K), R15.2
- no-connect marks 9 -> 8
Other:
- moved on the sheet: D1, D10, D11, D12, D13, D14, D15, D16, D17, D18, D2, D3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
